File: rpi_hat.kicad_sch (KiCad schematic)
At the start: 10 parts, among them U1 RASPBERRY_PI_3_MODEL_B+

Commit message: hat changes in design and ideation
Parts:
- U1: footprint Module:Raspberry_Pi_Zero_Socketed_THT_FaceDown_MountingHoles -> MODULE_RASPBERRY_PI_3_MODEL_B+:MODULE_RASPBERRY_PI_3_MODEL_B+
Connections:
- net 3v3: now also D4.1 (VDD), D5.1 (VDD), D6.1 (VDD), D7.1 (VDD), D8.1 (VDD), D9.1 (VDD), U1.2 (5V0), U1.4 (5V0); no longer U1.1 (3V3), U1.17 (3V3)
- new net: U1.1 (3V3), U1.17 (3V3)
Other:
- moved on the sheet: D4, D5, D6, D8, D9
